File: circuitoKicad/ShieldEduIfspSTM32.kicad_pcb (KiCad board)
At the start: 2 copper layers, 100 x 75 mm, 84 parts, among them J1 VIM, J10 OUTPUT, J11 OUT-MUX, J2 I2C, J3 I2C, J4 Bluetooth_UsbSerial, J5 USART_1B, J6 SPI, J7 ADC, J8 USB / CAM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

Commit message: REV160
Parts:
- removed JP2: JUMP3, Connector_PinSocket_2.54mm:PinSocket_1x03_P2.54mm_Vertical
- moved J4 4.47 mm to (145.0, 73.8)
Connections:
- J2 pad 3: /VCOM -> +5V
- J3 pad 3: /VCOM -> +5V
- J5 pad 3: /VCOM -> +5V
- J7 pad 3: /VCOM -> +5V
- J8 pad 3: /VCOM -> +5V
Routing:
- net /VCOM: track 82.6 -> 0.00 mm, vias 1 -> 0
- net /PA9: track 39.4 -> 71.6 mm, vias 1 -> 0
- net +5V: track 311.7 -> 328.5 mm, vias 4 -> 3
- net +3V3: track 292.6 -> 282.5 mm
- net /PA10: track 44.0 -> 53.5 mm, vias 2 -> 1
Other:
- board text added: "PWR OUT 5V"
- board text added: "SHIELD EDU IFSP STM32 2019 REV1.60 Pedro Igor Borçatti da Silva Rogerio Daniel Dantas"
- board text removed: "SHIELD EDU IFSP STM32 2019 REV1.50 Pedro Igor Borçatti da Silva Rogerio Daniel Dantas"
- board text removed: "VCOM PWR OUT 3V3-5V"
