File: circuitoKicad/ShieldEduIfspSTM32.sch (KiCad schematic (older format))
At the start: 26 parts, among them J1 VIM, J10 OUTPUT, J11 OUT-MUX, J2 I2C, J3 I2C, J4 Bluetooth_UsbSerial, J5 USART_1B, J6 SPI, J7 ADC, J8 USB / CAM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

Commit message: REV160
Parts:
- removed JP2: JUMP3, Connector_PinSocket_2.54mm:PinSocket_1x03_P2.54mm_Vertical, symbol MyLib-ALL:JUMP3
Connections:
- net VCOM is gone; now on net +5V: J2.3 (Pin_3), J3.3 (Pin_3), J5.3 (Pin_3), J7.3 (Pin_3), J8.3 (Pin_3)
- net PA0: now also R2.2, R3.1
Other:
- note removed: "Seletor de tensão para\nsaídas modulares"
Changed lines of the file:
@@
 Sheet 1 3
 Title "SHIELD EDU IFSP STM32"
-Date "2019-07-25"
-Rev "1.5"
+Date "2019-07-29"
+Rev "1.6"
 Comp "SHIELD EDU"
 Comment1 "ATENÇÃO há pinos com Tolerância a 5V no entendo não TODOS "
@@
 	0    -1   -1   0
 $EndComp
-$Comp
-L power:+3V3 #PWR0104
-U 1 1 5D6CA56B
-P 7600 3200
-AR Path="/5D6CA56B" Ref="#PWR0104"  Part="1"
-AR Path="/5D49BDAC/5D6CA56B" Ref="#PWR?"  Part="1"
-F 0 "#PWR0104" H 7600 3050 50  0001 C CNN
-F 1 "+3V3" V 7600 3450 50  0000 C CNN
-F 2 "" H 7600 3200 50  0001 C CNN
-F 3 "" H 7600 3200 50  0001 C CNN
-	1    7600 3200
-	-1   0    0    -1
-$EndComp
 Wire Wire Line
 	8450 1500 8450 1300
@@
 Wire Wire Line
 	9800 3200 9800 3100
-Wire Wire Line
-	7600 3200 7600 3300
 $Comp
 L Device:R R?
@@
 	1    0    0    -1
 $EndComp
-Text Label 9450 1500 3    39   ~ 0
-VCOM
-Text Label 8950 1500 3    39   ~ 0
-VCOM
-Text Label 8450 1500 3    39   ~ 0
-VCOM
-Wire Wire Line
-	7600 3900 7600 3800
-Wire Wire Line
-	7450 3550 7500 3550
-Text Label 7450 3550 2    39   ~ 0
-VCOM
 $Comp
 L power:+5V #PWR0110
 U 1 1 5D6CA5FA
-P 7600 3900
+P 8450 1500
 AR Path="/5D6CA5FA" Ref="#PWR0110"  Part="1"
 AR Path="/5D49BDAC/5D6CA5FA" Ref="#PWR?"  Part="1"
-F 0 "#PWR0110" H 7600 3750 50  0001 C CNN
-F 1 "+5V" V 7600 4100 50  0000 C CNN
-F 2 "" H 7600 3900 50  0001 C CNN
-F 3 "" H 7600 3900 50  0001 C CNN
-	1    7600 3900
+F 0 "#PWR0110" H 8450 1350 50  0001 C CNN
+F 1 "+5V" V 8450 1700 50  0000 C CNN
+F 2 "" H 8450 1500 50  0001 C CNN
+F 3 "" H 8450 1500 50  0001 C CNN
+	1    8450 1500
 	1    0    0    1
 $EndComp
@@
 Text Notes 7050 700  0    59   ~ 12
 Saída  M2M / GPIO Externa Modular
-$Comp
-L MyLib-ALL:JUMP3 JP?
-U 1 1 5D6CA610
-P 7600 3550
-AR Path="/5D49BDAC/5D6CA610" Ref="JP?"  Part="1"
-AR Path="/5D6CA610" Ref="JP2"  Part="1"
-F 0 "JP2" H 7600 3659 50  0000 C CNN
-F 1 "JUMP3" H 7600 3750 50  0000 C CNN
-F 2 "Connector_PinSocket_2.54mm:PinSocket_1x03_P2.54mm_Vertical" H 7600 3550 50  0001 C CNN
-F 3 "" H 7600 3550 50  0000 C CNN
-	1    7600 3550
-	0    1    1    0
-$EndComp
 $Comp
 L power:Earth #PWR0111
@@
 Wire Wire Line
 	8350 2350 8350 2250
-Text Label 8450 2450 3    39   ~ 0
-VCOM
 $Comp
 L Connector_Generic:Conn_01x04 J?
@@
 Wire Wire Line
 	9850 1400 9850 1300
-Text Label 9950 1500 3    39   ~ 0
-VCOM
 $Comp
 L Connector_Generic:Conn_01x06 J?
@@
 	-1   0    0    1
 $EndComp
-Text Label 9150 3550 2    47   ~ 0
+Text Label 8950 3550 2    47   ~ 0
 PA0
 Text Label 9650 3550 2    47   ~ 0
@@
 Text Notes 10250 4150 1    47   ~ 0
 ADC 12 Bits\nTOLERÂNCIA DO PINO 3V3\nCOM DIVISOR 0V A 30V
-Text Notes 8050 4150 1    47   ~ 0
-Seletor de tensão para\nsaídas modulares
 Text Notes 1600 1600 0    47   ~ 0
 3V3 500mA\n1650mW
@@
 Text Notes 5150 4250 0    47   ~ 0
 VBAT, C12, C15 estão dedicados \npara clock (cristal externo) do RTC do ARM
+$Comp
+L power:+5V #PWR0104
+U 1 1 5D40E44A
+P 8950 1500
+AR Path="/5D40E44A" Ref="#PWR0104"  Part="1"
+AR Path="/5D49BDAC/5D40E44A" Ref="#PWR?"  Part="1"
+F 0 "#PWR0104" H 8950 1350 50  0001 C CNN
+F 1 "+5V" V 8950 1700 50  0000 C CNN
+F 2 "" H 8950 1500 50  0001 C CNN
+F 3 "" H 8950 1500 50  0001 C CNN
+	1    8950 1500
+	1    0    0    1
+$EndComp
+$Comp
+L power:+5V #PWR0123
+U 1 1 5D40E487
+P 9450 1500
+AR Path="/5D40E487" Ref="#PWR0123"  Part="1"
+AR Path="/5D49BDAC/5D40E487" Ref="#PWR?"  Part="1"
+F 0 "#PWR0123" H 9450 1350 50  0001 C CNN
+F 1 "+5V" V 9450 1700 50  0000 C CNN
+F 2 "" H 9450 1500 50  0001 C CNN
+F 3 "" H 9450 1500 50  0001 C CNN
+	1    9450 1500
+	1    0    0    1
+$EndComp
+$Comp
+L power:+5V #PWR0124
+U 1 1 5D40E4C4
+P 8450 2450
+AR Path="/5D40E4C4" Ref="#PWR0124"  Part="1"
+AR Path="/5D49BDAC/5D40E4C4" Ref="#PWR?"  Part="1"
+F 0 "#PWR0124" H 8450 2300 50  0001 C CNN
+F 1 "+5V" V 8450 2650 50  0000 C CNN
+F 2 "" H 8450 2450 50  0001 C CNN
+F 3 "" H 8450 2450 50  0001 C CNN
+	1    8450 2450
+	1    0    0    1
+$EndComp
+$Comp
+L power:+5V #PWR0125
+U 1 1 5D40EDBA
+P 9950 1500
+AR Path="/5D40EDBA" Ref="#PWR0125"  Part="1"
+AR Path="/5D49BDAC/5D40EDBA" Ref="#PWR?"  Part="1"
+F 0 "#PWR0125" H 9950 1350 50  0001 C CNN
+F 1 "+5V" V 9950 1700 50  0000 C CNN
+F 2 "" H 9950 1500 50  0001 C CNN
+F 3 "" H 9950 1500 50  0001 C CNN
+	1    9950 1500
+	1    0    0    1
+$EndComp
 $EndSCHEMATC
